File: negative-voltage/NegativeVoltage.kicad_pcb (KiCad board)
At the start: 2 copper layers, 11 parts, among them J1 Screw_Terminal_01x02, J2 Screw_Terminal_01x02, U1 LM555

Commit message: Initial routing
Parts:
- moved J2 50.8 mm to (99.1, 116.8), turned to 90 degrees
- moved D2 49.7 mm to (77.5, 129.5)
- moved C3 47.8 mm to (61.0, 121.9), turned to 90 degrees
- moved D1 46.0 mm to (68.6, 120.7), turned to 270 degrees
- moved C4 39.4 mm to (91.4, 125.7), turned to 90 degrees
- moved J1 20.1 mm to (55.9, 113.0), turned to 90 degrees
- moved R1 16.7 mm to (64.8, 100.3)
- moved C2 11.7 mm to (68.6, 110.5), turned to 180 degrees
- moved C1 5.24 mm to (83.8, 120.7), turned to 180 degrees
- moved R2 4.58 mm to (90.2, 106.7)
- moved U1 2.54 mm to (72.4, 106.7)
Routing:
- net GND: track 0.00 -> 70.7 mm
- net VCC: track 0.00 -> 56.4 mm
- net N$3: track 0.00 -> 31.6 mm
- net N$1: track 0.00 -> 24.8 mm
- net N$6: track 0.00 -> 21.2 mm
- net N$4: track 0.00 -> 20.7 mm
- net N$5: track 0.00 -> 19.7 mm
- net N$2: track 0.00 -> 7.93 mm
Other:
- board outline added: 53.3 x 69.9 mm
