File: eeprom-programmer/hardware/EEPROMBoard.kicad_pcb (KiCad board)
At the start: 2 copper layers, 17 parts, among them J1 Conn_02x03_Odd_Even, J2 Conn_01x03, J3 DB9_Female, J4 Conn_01x06, J5 Conn_01x06, U1 MAX232, U2 28C256, U3 ATtiny2313V-10PU, U4 74HC595, U5 74HC595

Commit message: PCB layout finished... Will it really work?
Parts:
- removed C2, C3, C4: 1uF, Capacitor_THT:CP_Radial_D5.0mm_P2.50mm
- removed C5: C, Capacitor_THT:C_Disc_D4.3mm_W1.9mm_P5.00mm
- removed J4, J5: Conn_01x06, Connector_PinHeader_2.54mm:PinHeader_1x06_P2.54mm_Vertical
- removed U5: 74HC595, Package_DIP:DIP-16_W7.62mm
- C1: value 1uF -> 10u; footprint Capacitor_THT:CP_Radial_D5.0mm_P2.50mm -> Capacitor_THT:C_Disc_D4.3mm_W1.9mm_P5.00mm
- J2: value Conn_01x03 -> Screw_Terminal_01x02; footprint Connector_BarrelJack:BarrelJack_CUI_PJ-102AH_Horizontal -> TerminalBlock:TerminalBlock_bornier-2_P5.08mm
- J3: value DB9_Female -> Conn_01x06; footprint Connector_Dsub:DSUB-9_Female_Horizontal_P2.77x2.84mm_EdgePinOffset7.70mm_Housed_MountingHolesOffset9.12mm -> Connector_PinHeader_2.54mm:PinHeader_1x06_P2.54mm_Vertical
- R1: value R -> 10k
- U1: value MAX232 -> 28C256; footprint Package_DIP:DIP-16_W7.62mm -> Socket:DIP_Socket-28_W11.9_W12.7_W15.24_W17.78_W18.5_3M_228-1277-00-0602J
- U2: value 28C256 -> ATtiny2313V-10PU; footprint Socket:DIP_Socket-28_W11.9_W12.7_W15.24_W17.78_W18.5_3M_228-1277-00-0602J -> Package_DIP:DIP-20_W7.62mm_Socket_LongPads
- U3: value ATtiny2313V-10PU -> 74HC595; footprint Package_DIP:DIP-20_W7.62mm -> Package_DIP:DIP-16_W7.62mm_Socket_LongPads
- U4: footprint Package_DIP:DIP-16_W7.62mm -> Package_DIP:DIP-16_W7.62mm_Socket_LongPads
- moved C1 113.5 mm to (99.5, 66.8), turned to 180 degrees
- moved D1 79.8 mm to (108.4, 48.0), turned to 180 degrees
- moved R1 76.2 mm to (107.5, 55.7), turned to 180 degrees
- moved J1 70.1 mm to (98.8, 81.9), turned to 180 degrees
- moved J2 54.5 mm to (94.7, 55.9), turned to 270 degrees
- moved J3 53.4 mm to (96.7, 92.8)
- moved U3 37.2 mm to (170.1, 82.7)
- moved U2 22.6 mm to (111.8, 86.8)
- moved U1 19.0 mm to (137.8, 61.3)
- moved U4 17.6 mm to (119.4, 73.7), turned to 180 degrees
Connections:
- C1 pad 1: N$26 -> N$27
- C1 pad 2: N$27 -> GND
- D1 pad 2: N$35 -> N$27
- J1 pad 1: DATA_BUS6 -> DATA_BUS1
- J1 pad 3: DATA_BUS7 -> DATA_BUS0
- J1 pad 4: DATA_BUS5 -> DATA_BUS2
- J1 pad 5: N$35 -> N$27
- J3 pad 1: (no net) -> GND
- J3 pad 2: N$32 -> (no net)
- J3 pad 3: N$33 -> N$24
- J3 pad 5: GND -> N$25
- J3 pad 6: (no net) -> VCC
- R1 pad 2: N$35 -> N$27
- U1 pad 1: N$26 -> ADDRESS_BUS14
- U1 pad 10: (no net) -> ADDRESS_BUS0
- U1 pad 11: N$24 -> DATA_BUS0
- U1 pad 12: N$25 -> DATA_BUS1
- U1 pad 13: N$33 -> DATA_BUS2
- U1 pad 14: N$32 -> GND
- U1 pad 15: GND -> DATA_BUS3
- U1 pad 16: VCC -> DATA_BUS4
- U1 pad 2: N$31 -> ADDRESS_BUS12
- U1 pad 3: N$27 -> ADDRESS_BUS7
- U1 pad 4: N$28 -> ADDRESS_BUS6
- U1 pad 5: N$29 -> ADDRESS_BUS5
- U1 pad 6: N$30 -> ADDRESS_BUS4
- U1 pad 7: (no net) -> ADDRESS_BUS3
- U1 pad 8: (no net) -> ADDRESS_BUS2
- U1 pad 9: (no net) -> ADDRESS_BUS1
- U2 pad 1: ADDRESS_BUS14 -> N$27
- U2 pad 10: ADDRESS_BUS0 -> GND
- U2 pad 11: DATA_BUS0 -> ADDR_RCLK
- U2 pad 12: DATA_BUS1 -> DATA_BUS7
- U2 pad 13: DATA_BUS2 -> DATA_BUS6
- U2 pad 14: GND -> DATA_BUS5
- U2 pad 15: DATA_BUS3 -> DATA_BUS4
- U2 pad 16: DATA_BUS4 -> DATA_BUS3
- U2 pad 17: DATA_BUS5 -> DATA_BUS2
- U2 pad 18: DATA_BUS6 -> DATA_BUS1
- U2 pad 19: DATA_BUS7 -> DATA_BUS0
- U2 pad 2: ADDRESS_BUS12 -> N$24
- U2 pad 20: GND -> VCC
- U2 pad 3: ADDRESS_BUS7 -> N$25
- U2 pad 4: ADDRESS_BUS6 -> (no net)
- U2 pad 5: ADDRESS_BUS5 -> (no net)
- U2 pad 6: ADDRESS_BUS4 -> ADDR_OUTPUT
- U2 pad 7: ADDRESS_BUS3 -> ADDR_SRCLK
- U2 pad 8: ADDRESS_BUS2 -> ~EEPROM_OE
- U2 pad 9: ADDRESS_BUS1 -> ~EEPROM_WE
- U3 pad 1: N$35 -> ADDRESS_BUS9
- U3 pad 10: GND -> VCC
- U3 pad 11: ADDR_RCLK -> ADDR_SRCLK
- U3 pad 12: DATA_BUS0 -> ADDR_RCLK
- U3 pad 13: DATA_BUS1 -> GND
- U3 pad 14: DATA_BUS2 -> N$26
- U3 pad 15: DATA_BUS3 -> ADDRESS_BUS8
- U3 pad 16: DATA_BUS4 -> VCC
- U3 pad 2: N$25 -> ADDRESS_BUS10
- U3 pad 3: N$24 -> ADDRESS_BUS11
- U3 pad 4: (no net) -> ADDRESS_BUS12
- U3 pad 5: (no net) -> ADDRESS_BUS13
- U3 pad 6: ADDR_OUTPUT -> ADDRESS_BUS14
- U3 pad 7: ADDR_SRCLK -> (no net)
- U3 pad 8: ~EEPROM_OE -> GND
- U3 pad 9: ~EEPROM_WE -> (no net)
- U4 pad 1: ADDRESS_BUS9 -> ADDRESS_BUS1
- U4 pad 14: N$34 -> ADDR_OUTPUT
- U4 pad 15: ADDRESS_BUS8 -> ADDRESS_BUS0
- U4 pad 2: ADDRESS_BUS10 -> ADDRESS_BUS2
- U4 pad 3: ADDRESS_BUS11 -> ADDRESS_BUS3
- U4 pad 4: ADDRESS_BUS12 -> ADDRESS_BUS4
- U4 pad 5: ADDRESS_BUS13 -> ADDRESS_BUS5
- U4 pad 6: ADDRESS_BUS14 -> ADDRESS_BUS6
- U4 pad 7: (no net) -> ADDRESS_BUS7
- U4 pad 9: (no net) -> N$26
Routing:
- net VCC: track 0.00 -> 279.8 mm, vias 0 -> 12
- net GND: track 0.00 -> 234.1 mm, vias 0 -> 2
- net ADDR_RCLK: track 0.00 -> 158.3 mm, vias 0 -> 6
- net ADDR_SRCLK: track 0.00 -> 145.3 mm, vias 0 -> 5
- net ~EEPROM_OE: track 0.00 -> 142.8 mm, vias 0 -> 4
- net ~EEPROM_WE: track 0.00 -> 125.3 mm, vias 0 -> 4
- net N$26: track 0.00 -> 109.8 mm, vias 0 -> 2
- net DATA_BUS2: track 0.00 -> 76.1 mm, vias 0 -> 4
- net ADDRESS_BUS14: track 0.00 -> 71.4 mm, vias 0 -> 2
- net ADDRESS_BUS12: track 0.00 -> 64.8 mm, vias 0 -> 2
- net DATA_BUS7: track 0.00 -> 60.0 mm
- net DATA_BUS6: track 0.00 -> 54.5 mm
- net N$27: track 0.00 -> 51.4 mm, vias 0 -> 3
- net DATA_BUS0: track 0.00 -> 50.1 mm, vias 0 -> 2
- net DATA_BUS1: track 0.00 -> 49.9 mm, vias 0 -> 2
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Other:
- net class Default: clearance 0.2 -> 0.3; trace_width 0.25 -> 0.3; via_dia 0.8 -> 1.5; via_drill 0.6 -> 0.8
- net class Power added: clearance 0.3, trace_width 0.4, via_dia 1.5, via_drill 0.8
- rule trace_clearance: 0.2 -> 0.3

Commit message: Not sure what changed
Routing:
- net ADDR_SRCLK: track 145.3 -> 148.6 mm
- added copper zone on B.Cu, net (none)
- added copper zone on F.Cu, net (none)
- added copper zone on B.Cu, net GND
- added copper zone on F.Cu, net GND
Other:
- board outline added: 98.8 x 69.9 mm
